File: SchiitBox.kicad_pcb (KiCad board)
At the start: 2 copper layers, 122 x 84 mm, 21 parts, among them J1 AudioJack4dpb

Commit message: updated board trace, added debounce circuits
Parts:
- removed the ? at (108.5, 82.0)
- removed the ? at (128.7, 82.0)
- removed the ? at (103.5, 82.0)
- removed the ? at (133.7, 82.0)
- removed the ? at (131.2, 82.0)
- removed the ? at (126.2, 82.0)
- removed the ? at (106.0, 82.0)
- removed the ? at (101.0, 82.0)
- added ?: , , F.Cu at (133.9, 82.0)
- added ?: , , F.Cu at (126.2, 82.0)
- added ?: , , F.Cu at (103.6, 82.0)
- added ?: , , F.Cu at (128.8, 82.0)
- added ?: , , F.Cu at (106.1, 82.0)
- added ?: , , F.Cu at (131.3, 82.0)
- added ?: , , F.Cu at (101.0, 82.0)
- added ?: , , F.Cu at (108.7, 82.0)
- added REF**: R1, Resistor_SMD:R_0603_1608Metric_Pad0.98x0.95mm_HandSolder, F.Cu at (124.3, 63.5)
- added REF**: R1, Resistor_SMD:R_0603_1608Metric_Pad0.98x0.95mm_HandSolder, F.Cu at (124.3, 65.9)
- added REF**: R1, Capacitor_SMD:C_1206_3216Metric_Pad1.33x1.80mm_HandSolder, F.Cu at (106.9, 50.2)
- added REF**: 42 (10k), Resistor_SMD:R_0603_1608Metric_Pad0.98x0.95mm_HandSolder, F.Cu at (124.3, 61.1)
- added REF**: R2, Capacitor_SMD:C_1206_3216Metric_Pad1.33x1.80mm_HandSolder, F.Cu at (113.8, 50.3)
- added REF**: R2, Resistor_SMD:R_0603_1608Metric_Pad0.98x0.95mm_HandSolder, F.Cu at (124.3, 58.6)
- added REF**: R2, Resistor_SMD:R_0603_1608Metric_Pad0.98x0.95mm_HandSolder, F.Cu at (124.3, 56.2)
- added REF**: R2, Resistor_SMD:R_0603_1608Metric_Pad0.98x0.95mm_HandSolder, F.Cu at (124.3, 53.7)
- added REF**: 104k (.1u), Capacitor_SMD:C_1206_3216Metric_Pad1.33x1.80mm_HandSolder, F.Cu at (117.3, 50.3)
- added REF**: R2, Capacitor_SMD:C_1206_3216Metric_Pad1.33x1.80mm_HandSolder, F.Cu at (110.4, 50.2)
- added REF**: R1, Capacitor_SMD:C_1206_3216Metric_Pad1.33x1.80mm_HandSolder, F.Cu at (103.4, 50.2)
- added REF**: R1, Capacitor_SMD:C_1206_3216Metric_Pad1.33x1.80mm_HandSolder, F.Cu at (100.0, 50.1)
- turned ? to 90 degrees (x2)
Connections:
- REF** pad : 3V3 -> GPIO_0
Routing:
- net 3V3: track 0.00 -> 70.2 mm
- net clk_2: track 0.00 -> 49.9 mm
- net dt_2: track 0.00 -> 48.1 mm
- net sw_2: track 0.00 -> 45.8 mm
- net clk_1: track 0.00 -> 37.8 mm
- net dt_1: track 0.00 -> 35.9 mm
- net sw_1: track 0.00 -> 33.9 mm
Other:
- board size 122 x 84 mm -> 122 x 86.1 mm

Commit message: finalized SchiitBox design
Parts:
- added ?: , , F.Cu at (57.9, 102.4)
- added ?: , , F.Cu at (89.2, 102.4)
- turned ? to 180 degrees
Connections:
- REF** pad : dt_2 -> GPIO_2
- REF** pad : sw_2 -> GPIO_0
- REF** pad : GPIO_13 -> gnd
- REF** pad : GPIO_0 -> 3V3
- REF** pad : sw_1 -> GPIO_12
- REF** pad : dt_1 -> GPIO_13
- REF** pad : clk_1 -> GPIO_14
- REF** pad : gnd -> GPIO_12
Routing:
- net GPIO_0: track 0.00 -> 97.8 mm, vias 0 -> 1
- net GPIO_2: track 0.00 -> 95.9 mm, vias 0 -> 1
- net GPIO_3: track 0.00 -> 93.5 mm, vias 0 -> 1
- net GPIO_12: track 0.00 -> 72.4 mm, vias 0 -> 1
- net GPIO_13: track 0.00 -> 70.0 mm, vias 0 -> 1
- net GPIO_14: track 0.00 -> 68.1 mm, vias 0 -> 1
- net clk_2: track 49.9 -> 0.00 mm
- net dt_2: track 48.1 -> 0.00 mm
- net sw_2: track 45.8 -> 0.00 mm
- net clk_1: track 37.8 -> 0.00 mm
- net dt_1: track 35.9 -> 0.00 mm
- net sw_1: track 33.9 -> 0.00 mm
Other:
- board size 122 x 86.1 mm -> 122 x 85.4 mm
